File: TPIC6B595_power_sift_reg_breakout/board.kicad_pcb (KiCad board)
At the start: 2 copper layers, 49.5 x 53.3 mm, 5 parts, among them IC1 DIL20, J1 CONN_01X08, J2 CONN_01X06, J3 CONN_01X06

Commit message: misc work on PCB design
Parts:
- added J4: CONN_01X01, Pin_Headers:Pin_Header_Straight_1x01_Pitch2.54mm, F.Cu at (248.9, 127.0)
- added J5: CONN_02X08, Pin_Headers:Pin_Header_Straight_2x08_Pitch2.54mm, F.Cu at (207.0, 121.9)
- added J6: CONN_02X08, Pin_Headers:Pin_Header_Straight_2x08_Pitch2.54mm, F.Cu at (212.1, 121.9)
- added J8: HEADER_8, Connectors_Phoenix:PhoenixContact_MCV-GF_08x5.08mm_Vertical_ThreadedFlange, F.Cu at (226.1, 111.8)
- moved R1 21.7 mm to (193.0, 152.4)
- moved J1 6.35 mm to (218.4, 121.9)
- moved J2 4.58 mm to (196.8, 109.2)
- moved IC1 4.58 mm to (185.4, 119.4)
- moved J3 3.81 mm to (209.6, 153.7)
Connections:
- J1 pad 1: /DRAIN_7 -> /DRAIN_0
- J1 pad 2: /DRAIN_6 -> /DRAIN_1
- J1 pad 3: /DRAIN_5 -> /DRAIN_7
- J1 pad 4: /DRAIN_4 -> /DRAIN_6
- J1 pad 5: /DRAIN_3 -> /DRAIN_5
- J1 pad 6: /DRAIN_2 -> /DRAIN_4
- J1 pad 7: /DRAIN_1 -> /DRAIN_2
- J1 pad 8: /DRAIN_0 -> /DRAIN_3
Routing:
- net /DRAIN_0: track 0.00 -> 72.4 mm
- net /DRAIN_2: track 0.00 -> 64.6 mm
- net GND: track 0.00 -> 46.6 mm
- net +5V: track 74.9 -> 112.2 mm, vias 0 -> 2
- net /SER_OUT: track 35.6 -> 56.2 mm
- net /en: track 85.1 -> 68.6 mm
- net /DRAIN_1: track 81.3 -> 67.8 mm
- net /SER_IN: track 19.4 -> 31.7 mm
- net /SRCLR: track 31.8 -> 22.9 mm, vias 2 -> 0
- net /DRAIN_4: track 29.3 -> 34.8 mm
- net /SRCK: track 74.9 -> 80.0 mm
- net /DRAIN_5: track 29.3 -> 33.0 mm
- net /DRAIN_7: track 33.0 -> 36.6 mm
- net /DRAIN_6: track 33.0 -> 35.6 mm
- net /RCK: track 70.1 -> 67.6 mm
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Other:
- outline, holes or cut-outs redrawn
- board text added: "Shift Register of DOOM"
- board text added: "https://github.com/busyDuckman/ShiftRegisterOfDoom"
